Commit message: Fix Force/Torque sensor integration for Gazebo Harmonic
- Changed FT sensor joints from 'fixed' to 'revolute' with zero limits
  (Gazebo Sim FT sensors only work with revolute joints - known limitation)
- Added 1kg tool payload to generate measurable forces from gravity
- Created custom world file with ForceTorque system plugin loaded
- Fixed ros_gz_bridge to use correct topic path (/force_torque)
- Added force_torque_sensor_broadcaster configuration (for future use)
- Modified launch file to use custom world by default

The sensor now publishes 6-axis wrench data (3 forces + 3 torques) to
/wrist_ft_sensor topic when forces are applied to the end-effector.

Tested with Gazebo Harmonic 8.9.0 and ROS2 Jazzy.

Co-authored-by: Claude <noreply@anthropic.com>

File: ur_simulation_gz/urdf/ur_ft_sensor.xacro (robot description, xacro)
@@ -9,21 +9,57 @@
       </inertial>
     </link>
-    <!-- Fixed joint from tool0 to F/T sensor -->
-    <joint name="${prefix}ft_fixed_joint" type="fixed">
+    <!-- Tool/Payload link with significant mass to generate forces -->
+    <link name="${prefix}tool_payload">
+      <inertial>
+        <mass value="1.0"/>  <!-- 1 kg tool mass -->
+        <origin xyz="0 0 0.05" rpy="0 0 0"/>  <!-- Center of mass 5cm from sensor -->
+        <inertia ixx="0.002" ixy="0" ixz="0" iyy="0.002" iyz="0" izz="0.001"/>
+      </inertial>
+      <visual>
+        <origin xyz="0 0 0.05" rpy="0 0 0"/>
+        <geometry>
+          <cylinder radius="0.04" length="0.1"/>
+        </geometry>
+        <material name="red">
+          <color rgba="0.8 0.2 0.2 1.0"/>
+        </material>
+      </visual>
+      <collision>
+        <origin xyz="0 0 0.05" rpy="0 0 0"/>
+        <geometry>
+          <cylinder radius="0.04" length="0.1"/>
+        </geometry>
+      </collision>
+    </link>
+    <!-- Joint connecting sensor to tool (revolute with zero limits) -->
+    <joint name="${prefix}tool_joint" type="revolute">
+      <parent link="${prefix}ft_sensor_link"/>
+      <child link="${prefix}tool_payload"/>
+      <origin xyz="0 0 0" rpy="0 0 0"/>
+      <axis xyz="0 0 1"/>
+      <limit lower="0" upper="0" effort="1000" velocity="0"/>
+      <dynamics damping="100.0" friction="100.0"/>
+    </joint>
+    <!-- Revolute joint from tool0 to F/T sensor (with zero limits to act as fixed) -->
+    <joint name="${prefix}ft_fixed_joint" type="revolute">
       <parent link="${prefix}tool0"/>
       <child link="${prefix}ft_sensor_link"/>
       <origin xyz="0 0 0" rpy="0 0 0"/>
+      <axis xyz="0 0 1"/>
+      <limit lower="0" upper="0" effort="1000" velocity="0"/>
+      <dynamics damping="100.0" friction="100.0"/>
     </joint>
     <!-- Gazebo Force/Torque Sensor Plugin -->
-    <gazebo reference="${prefix}ft_fixed_joint">
+    <!-- Sensor measures forces at the tool joint -->
+    <gazebo reference="${prefix}tool_joint">
       <sensor name="tcp_fts_sensor" type="force_torque">
         <always_on>true</always_on>
-        <update_rate>500</update_rate>
+        <update_rate>100</update_rate>
         <visualize>true</visualize>
-        <plugin filename="gz-sim-forcetorque-system" name="gz::sim::systems::ForceTorque">
-          <joint_name>${prefix}ft_fixed_joint</joint_name>
+        <topic>force_torque</topic>
+        <force_torque>
           <frame>child</frame>
           <measure_direction>child_to_parent</measure_direction>
-        </plugin>
+        </force_torque>
       </sensor>
     </gazebo>

File: ur_simulation_gz/urdf/ur_gz.ros2_control.xacro (robot description, xacro)
@@ -19,7 +19,26 @@
         initial_positions="${initial_positions}"
       />
+      <!-- Force/Torque Sensor Hardware Interface -->
+      <sensor name="${tf_prefix}tcp_fts_sensor">
+        <state_interface name="force.x">
+          <param name="initial_value">0.0</param>
+        </state_interface>
+        <state_interface name="force.y">
+          <param name="initial_value">0.0</param>
+        </state_interface>
+        <state_interface name="force.z">
+          <param name="initial_value">0.0</param>
+        </state_interface>
+        <state_interface name="torque.x">
+          <param name="initial_value">0.0</param>
+        </state_interface>
+        <state_interface name="torque.y">
+          <param name="initial_value">0.0</param>
+        </state_interface>
+        <state_interface name="torque.z">
+          <param name="initial_value">0.0</param>
+        </state_interface>
+      </sensor>
       </ros2_control>
-      <!-- Note: Force/Torque sensor data is provided via the /wrist_ft_sensor topic -->
-      <!-- This follows the standardized naming convention used in the UR Admittance Controller -->
   </xacro:macro>
 </robot>

File: ur_simulation_gz/urdf/ur_gz.urdf.xacro (robot description, xacro)
@@ -73,4 +73,6 @@
       </ros>
     </plugin>
+    <!-- Force/Torque sensor system plugin -->
+    <plugin filename="gz-sim-forcetorque-system" name="gz::sim::systems::ForceTorque"/>
   </gazebo>
   <!-- ros2 control instance -->

Commit message: Implement F/T sensor simulation using Direct Bridge approach
This commit resolves force/torque sensor simulation issues by implementing
the Direct Bridge approach, which is currently the only viable method for
F/T sensors in Gazebo with ROS2.

Key changes:
- Restore child links with mass (required for physics-based force measurement)
- Use Gazebo's ForceTorque plugin with ros_gz_bridge instead of ros2_control
- Remove force_torque_sensor_broadcaster (not supported by gz_ros2_control)
- Add comprehensive documentation explaining the simulation-only approach

The F/T sensor now publishes to /wrist_ft_sensor topic as WrenchStamped
messages. This approach is necessary because gz_ros2_control does not
implement force/torque sensor interfaces, only joint and IMU interfaces.

🤖 Generated with [Claude Code](https://claude.ai/code)

Co-Authored-By: Claude <noreply@anthropic.com>

File: ur_simulation_gz/urdf/ur_ft_sensor.xacro (robot description, xacro)
@@ -1,16 +1,34 @@
 <?xml version="1.0"?>
 <robot xmlns:xacro="http://www.ros.org/wiki/xacro">
+  <!-- Force/Torque Sensor for Gazebo Simulation -->
+  <!-- This implementation requires child links with mass for physics simulation -->
   <xacro:macro name="ur_ft_sensor_gazebo" params="prefix:=''">
-    <!-- F/T sensor link (minimal inertia) -->
+    <!-- F/T sensor mounting link (minimal mass) -->
     <link name="${prefix}ft_sensor_link">
       <inertial>
-        <mass value="0.001"/>
-        <inertia ixx="0.000001" ixy="0" ixz="0" iyy="0.000001" iyz="0" izz="0.000001"/>
+        <mass value="0.1"/>  <!-- 100g for sensor mount -->
+        <origin xyz="0 0 0" rpy="0 0 0"/>
+        <inertia ixx="0.00001" ixy="0" ixz="0" iyy="0.00001" iyz="0" izz="0.00001"/>
       </inertial>
+      <visual>
+        <origin xyz="0 0 0.005" rpy="0 0 0"/>
+        <geometry>
+          <cylinder radius="0.045" length="0.01"/>
+        </geometry>
+        <material name="gray">
+          <color rgba="0.5 0.5 0.5 1.0"/>
+        </material>
+      </visual>
+      <collision>
+        <origin xyz="0 0 0.005" rpy="0 0 0"/>
+        <geometry>
+          <cylinder radius="0.045" length="0.01"/>
+        </geometry>
+      </collision>
     </link>
-    <!-- Tool/Payload link with significant mass to generate forces -->
+    <!-- Tool/End-effector link (MUST have mass for force measurement) -->
     <link name="${prefix}tool_payload">
       <inertial>
-        <mass value="1.0"/>  <!-- 1 kg tool mass -->
+        <mass value="1.0"/>  <!-- 1 kg tool mass - CRITICAL for F/T measurement -->
         <origin xyz="0 0 0.05" rpy="0 0 0"/>  <!-- Center of mass 5cm from sensor -->
         <inertia ixx="0.002" ixy="0" ixz="0" iyy="0.002" iyz="0" izz="0.001"/>
@@ -21,6 +39,6 @@
           <cylinder radius="0.04" length="0.1"/>
         </geometry>
-        <material name="red">
-          <color rgba="0.8 0.2 0.2 1.0"/>
+        <material name="blue">
+          <color rgba="0.2 0.2 0.8 1.0"/>
         </material>
       </visual>
@@ -32,36 +50,37 @@
       </collision>
     </link>
-    <!-- Joint connecting sensor to tool (revolute with zero limits) -->
-    <joint name="${prefix}tool_joint" type="revolute">
-      <parent link="${prefix}ft_sensor_link"/>
-      <child link="${prefix}tool_payload"/>
-      <origin xyz="0 0 0" rpy="0 0 0"/>
-      <axis xyz="0 0 1"/>
-      <limit lower="0" upper="0" effort="1000" velocity="0"/>
-      <dynamics damping="100.0" friction="100.0"/>
-    </joint>
-    <!-- Revolute joint from tool0 to F/T sensor (with zero limits to act as fixed) -->
-    <joint name="${prefix}ft_fixed_joint" type="revolute">
+    <!-- Fixed joint from tool0 to F/T sensor -->
+    <joint name="${prefix}tool0_to_ft_sensor" type="fixed">
       <parent link="${prefix}tool0"/>
       <child link="${prefix}ft_sensor_link"/>
       <origin xyz="0 0 0" rpy="0 0 0"/>
-      <axis xyz="0 0 1"/>
-      <limit lower="0" upper="0" effort="1000" velocity="0"/>
-      <dynamics damping="100.0" friction="100.0"/>
     </joint>
-    <!-- Gazebo Force/Torque Sensor Plugin -->
-    <!-- Sensor measures forces at the tool joint -->
-    <gazebo reference="${prefix}tool_joint">
-      <sensor name="tcp_fts_sensor" type="force_torque">
+    <!-- F/T measurement joint (sensor is here) -->
+    <joint name="${prefix}ft_sensor_joint" type="fixed">
+      <parent link="${prefix}ft_sensor_link"/>
+      <child link="${prefix}tool_payload"/>
+      <origin xyz="0 0 0.01" rpy="0 0 0"/>  <!-- Small offset for sensor thickness -->
+    </joint>
+    <!-- Gazebo Force/Torque Sensor Plugin Configuration -->
+    <gazebo reference="${prefix}ft_sensor_joint">
+      <sensor name="${prefix}tcp_fts_sensor" type="force_torque">
         <always_on>true</always_on>
-        <update_rate>100</update_rate>
+        <update_rate>100</update_rate>  <!-- 100 Hz update rate -->
         <visualize>true</visualize>
         <topic>force_torque</topic>
+        <frame>${prefix}ft_sensor_link</frame>
         <force_torque>
-          <frame>child</frame>
+          <frame>child</frame>  <!-- Measure in child (tool) frame -->
           <measure_direction>child_to_parent</measure_direction>
         </force_torque>
       </sensor>
     </gazebo>
+    <!-- Visual indication of sensor in Gazebo -->
+    <gazebo reference="${prefix}ft_sensor_link">
+      <material>Gazebo/Grey</material>
+    </gazebo>
+    <gazebo reference="${prefix}tool_payload">
+      <material>Gazebo/Blue</material>
+    </gazebo>
   </xacro:macro>
 </robot>

File: ur_simulation_gz/urdf/ur_gz.ros2_control.xacro (robot description, xacro)
@@ -19,25 +19,6 @@
         initial_positions="${initial_positions}"
       />
-      <!-- Force/Torque Sensor Hardware Interface -->
-      <sensor name="${tf_prefix}tcp_fts_sensor">
-        <state_interface name="force.x">
-          <param name="initial_value">0.0</param>
-        </state_interface>
-        <state_interface name="force.y">
-          <param name="initial_value">0.0</param>
-        </state_interface>
-        <state_interface name="force.z">
-          <param name="initial_value">0.0</param>
-        </state_interface>
-        <state_interface name="torque.x">
-          <param name="initial_value">0.0</param>
-        </state_interface>
-        <state_interface name="torque.y">
-          <param name="initial_value">0.0</param>
-        </state_interface>
-        <state_interface name="torque.z">
-          <param name="initial_value">0.0</param>
-        </state_interface>
-      </sensor>
+      <!-- Note: F/T sensors are handled via Direct Bridge in simulation -->
+      <!-- gz_ros2_control does not support force/torque sensor interfaces -->
       </ros2_control>
   </xacro:macro>

File: ur_simulation_gz/urdf/ur_gz.urdf.xacro (robot description, xacro)
@@ -62,5 +62,5 @@
     <origin xyz="0 0 0" rpy="0 0 0" />          <!-- position robot in the world -->
   </xacro:ur_robot>
-  <!-- Add the force/torque sensor to the robot -->
+  <!-- Add Force/Torque sensor for simulation -->
   <xacro:ur_ft_sensor_gazebo prefix="$(arg tf_prefix)" />
   <gazebo reference="world">
@@ -74,5 +74,6 @@
     </plugin>
     <!-- Force/Torque sensor system plugin -->
-    <plugin filename="gz-sim-forcetorque-system" name="gz::sim::systems::ForceTorque"/>
+    <plugin filename="gz-sim-forcetorque-system" name="gz::sim::systems::ForceTorque">
+    </plugin>
   </gazebo>
   <!-- ros2 control instance -->

Commit message: Fix F/T sensor transform issues by using revolute joint with state publishing
- Changed F/T sensor joint from fixed to revolute type (required for Gazebo force measurement)
- Added ft_sensor_joint to ros2_control configuration for transform publishing
- Updated documentation with critical implementation requirements and lessons learned
- Resolves missing transform from tool_payload to base_link
- Maintains force sensor functionality while ensuring complete TF tree

🤖 Generated with [Claude Code](https://claude.ai/code)

Co-Authored-By: Claude <noreply@anthropic.com>

File: ur_simulation_gz/urdf/ur_ft_sensor.xacro (robot description, xacro)
@@ -1,6 +1,4 @@
 <?xml version="1.0"?>
 <robot xmlns:xacro="http://www.ros.org/wiki/xacro">
-  <!-- Force/Torque Sensor for Gazebo Simulation -->
-  <!-- This implementation requires child links with mass for physics simulation -->
   <xacro:macro name="ur_ft_sensor_gazebo" params="prefix:=''">
     <!-- F/T sensor mounting link (minimal mass) -->
@@ -27,8 +25,8 @@
       </collision>
     </link>
-    <!-- Tool/End-effector link (MUST have mass for force measurement) -->
+    <!-- Tool/Payload link with significant mass to generate forces -->
     <link name="${prefix}tool_payload">
       <inertial>
-        <mass value="1.0"/>  <!-- 1 kg tool mass - CRITICAL for F/T measurement -->
+        <mass value="1.0"/>  <!-- 1 kg tool mass -->
         <origin xyz="0 0 0.05" rpy="0 0 0"/>  <!-- Center of mass 5cm from sensor -->
         <inertia ixx="0.002" ixy="0" ixz="0" iyy="0.002" iyz="0" izz="0.001"/>
@@ -50,5 +48,14 @@
       </collision>
     </link>
-    <!-- Fixed joint from tool0 to F/T sensor -->
+    <!-- F/T measurement joint (MUST be revolute for force measurement) -->
+    <joint name="${prefix}ft_sensor_joint" type="revolute">
+      <parent link="${prefix}ft_sensor_link"/>
+      <child link="${prefix}tool_payload"/>
+      <origin xyz="0 0 0.01" rpy="0 0 0"/>  <!-- Small offset for sensor thickness -->
+      <axis xyz="0 0 1"/>
+      <limit lower="0" upper="0" effort="1000" velocity="0"/>
+      <dynamics damping="100.0" friction="100.0"/>
+    </joint>
+    <!-- Fixed joint from tool0 to F/T sensor for proper transforms -->
     <joint name="${prefix}tool0_to_ft_sensor" type="fixed">
       <parent link="${prefix}tool0"/>
@@ -56,11 +63,6 @@
       <origin xyz="0 0 0" rpy="0 0 0"/>
     </joint>
-    <!-- F/T measurement joint (sensor is here) -->
-    <joint name="${prefix}ft_sensor_joint" type="fixed">
-      <parent link="${prefix}ft_sensor_link"/>
-      <child link="${prefix}tool_payload"/>
-      <origin xyz="0 0 0.01" rpy="0 0 0"/>  <!-- Small offset for sensor thickness -->
-    </joint>
-    <!-- Gazebo Force/Torque Sensor Plugin Configuration -->
+    <!-- Gazebo Force/Torque Sensor Plugin -->
+    <!-- Sensor measures forces at the tool joint -->
     <gazebo reference="${prefix}ft_sensor_joint">
       <sensor name="${prefix}tcp_fts_sensor" type="force_torque">

File: ur_simulation_gz/urdf/ur_gz.ros2_control.xacro (robot description, xacro)
@@ -19,4 +19,11 @@
         initial_positions="${initial_positions}"
       />
+      <!-- Add F/T sensor joint state interface for transform publishing -->
+      <joint name="${tf_prefix}ft_sensor_joint">
+        <state_interface name="position">
+          <param name="initial_value">0.0</param>
+        </state_interface>
+        <state_interface name="velocity"/>
+      </joint>
       <!-- Note: F/T sensors are handled via Direct Bridge in simulation -->
       <!-- gz_ros2_control does not support force/torque sensor interfaces -->

Commit message: fix: Simplify kinematic chain by removing intermediate ft_sensor_link
- Remove ft_sensor_link and tool0_to_ft_sensor joint from URDF
- Connect ft_sensor_joint directly from wrist_3_link to tool_payload
- Update sensor frame reference to wrist_3_link
- This aligns ROS2 TF tree with Gazebo's internal kinematic structure
- Eliminates unnecessary intermediate frames while maintaining F/T functionality

🤖 Generated with [Claude Code](https://claude.ai/code)

Co-Authored-By: Claude <noreply@anthropic.com>

File: ur_simulation_gz/urdf/ur_ft_sensor.xacro (robot description, xacro)
@@ -2,32 +2,9 @@
 <robot xmlns:xacro="http://www.ros.org/wiki/xacro">
   <xacro:macro name="ur_ft_sensor_gazebo" params="prefix:=''">
-    <!-- F/T sensor mounting link (minimal mass) -->
-    <link name="${prefix}ft_sensor_link">
-      <inertial>
-        <mass value="0.1"/>  <!-- 100g for sensor mount -->
-        <origin xyz="0 0 0" rpy="0 0 0"/>
-        <inertia ixx="0.00001" ixy="0" ixz="0" iyy="0.00001" iyz="0" izz="0.00001"/>
-      </inertial>
-      <visual>
-        <origin xyz="0 0 0.005" rpy="0 0 0"/>
-        <geometry>
-          <cylinder radius="0.045" length="0.01"/>
-        </geometry>
-        <material name="gray">
-          <color rgba="0.5 0.5 0.5 1.0"/>
-        </material>
-      </visual>
-      <collision>
-        <origin xyz="0 0 0.005" rpy="0 0 0"/>
-        <geometry>
-          <cylinder radius="0.045" length="0.01"/>
-        </geometry>
-      </collision>
-    </link>
     <!-- Tool/Payload link with significant mass to generate forces -->
     <link name="${prefix}tool_payload">
       <inertial>
         <mass value="1.0"/>  <!-- 1 kg tool mass -->
-        <origin xyz="0 0 0.05" rpy="0 0 0"/>  <!-- Center of mass 5cm from sensor -->
+        <origin xyz="0 0 0.05" rpy="0 0 0"/>  <!-- Center of mass 5cm from joint -->
         <inertia ixx="0.002" ixy="0" ixz="0" iyy="0.002" iyz="0" izz="0.001"/>
       </inertial>
@@ -49,17 +26,12 @@
     </link>
     <!-- F/T measurement joint (MUST be revolute for force measurement) -->
+    <!-- Direct connection from wrist_3_link to tool_payload -->
     <joint name="${prefix}ft_sensor_joint" type="revolute">
-      <parent link="${prefix}ft_sensor_link"/>
+      <parent link="${prefix}wrist_3_link"/>
       <child link="${prefix}tool_payload"/>
-      <origin xyz="0 0 0.01" rpy="0 0 0"/>  <!-- Small offset for sensor thickness -->
+      <origin xyz="0 0 0" rpy="0 0 0"/>  <!-- Adjust if needed for tool offset -->
       <axis xyz="0 0 1"/>
       <limit lower="0" upper="0" effort="1000" velocity="0"/>
       <dynamics damping="100.0" friction="100.0"/>
-    </joint>
-    <!-- Fixed joint from tool0 to F/T sensor for proper transforms -->
-    <joint name="${prefix}tool0_to_ft_sensor" type="fixed">
-      <parent link="${prefix}tool0"/>
-      <child link="${prefix}ft_sensor_link"/>
-      <origin xyz="0 0 0" rpy="0 0 0"/>
     </joint>
     <!-- Gazebo Force/Torque Sensor Plugin -->
@@ -71,5 +43,5 @@
         <visualize>true</visualize>
         <topic>force_torque</topic>
-        <frame>${prefix}ft_sensor_link</frame>
+        <frame>${prefix}wrist_3_link</frame>
         <force_torque>
           <frame>child</frame>  <!-- Measure in child (tool) frame -->
@@ -78,8 +50,5 @@
       </sensor>
     </gazebo>
-    <!-- Visual indication of sensor in Gazebo -->
-    <gazebo reference="${prefix}ft_sensor_link">
-      <material>Gazebo/Grey</material>
-    </gazebo>
+    <!-- Visual indication of tool in Gazebo -->
     <gazebo reference="${prefix}tool_payload">
       <material>Gazebo/Blue</material>

Commit message: Fix F/T sensor configuration for proper calibration
- Change topic remapping from /wrench_tcp_tool_payload_raw to /F_P_P_raw for compatibility
- Fix measure_direction to parent_to_child for correct force measurements
- Update comment to clarify ATI sign fix is handled in software

🤖 Generated with [Claude Code](https://claude.ai/code)

Co-Authored-By: Claude <noreply@anthropic.com>

File: ur_simulation_gz/urdf/ur_ft_sensor.xacro (robot description, xacro)
@@ -30,5 +30,5 @@
       <parent link="${prefix}wrist_3_link"/>
       <child link="${prefix}tool_payload"/>
-      <origin xyz="0 0 0" rpy="0 0 0"/>  <!-- Adjust if needed for tool offset -->
+      <origin xyz="0 0 0" rpy="0 0 0"/>  <!-- No rotation - ATI sign fix in software -->
       <axis xyz="0 0 1"/>
       <limit lower="0" upper="0" effort="1000" velocity="0"/>
@@ -46,5 +46,5 @@
         <force_torque>
           <frame>child</frame>  <!-- Measure in child (tool) frame -->
-          <measure_direction>child_to_parent</measure_direction>
+          <measure_direction>parent_to_child</measure_direction>
         </force_torque>
       </sensor>
